File: meshtastic_wio1262_v1.kicad_sch (KiCad schematic)
At the start: 59 parts, among them J1 SWDIO, SW1 SW_Push, U1 nRF52840, U2 Wio-SX1262, U3 BQ25185, U4 TPS61023, U5 WS-003DB, Y1 32.768kHz, Y3 32MHz

Commit message: add pdf schematic and update schematic
Parts:
- removed L8: 470nH, LCSC:IND-SMD_L2.0-W1.6_MHCHL201610A-1R0M-Q8A, symbol Device:L
- removed R5: 100kR, symbol Device:R
- removed U4: TPS61023, Package_TO_SOT_SMD:SOT-563, symbol 1_Custom_IC:TPS61023
- added C30, C31: 1uF, symbol 3_Custom_Semiconductors:Cap
- added J2: batt, symbol Connector:Conn_01x02_Socket
- added SW2, SW3: TS-1010-C-A, easyeda2kicad:KEY-SMD_TX-1010-X-X, symbol LCSC:TS-1010-C-A
- added U4: SSD1306 0.96 128*64, symbol 2_Custom_Module:SSD1306_Panel
- added U6: ATGM336H-5N31, easyeda2kicad:GPSM-SMD_ATGM336H-TR, symbol LCSC:ATGM336H-5N31
- added U7: TLV75533PDRV, Package_SON:WSON-6-1EP_2x2mm_P0.65mm_EP1x1.6mm, symbol Regulator_Linear:TLV75533PDRV
- C24: value 10uF -> 1uF; footprint (none) -> Capacitor_SMD:C_0603_1608Metric
- C25, C26: value 4.7uF -> 1uF; footprint (none) -> Capacitor_SMD:C_0603_1608Metric
- R4: value 453kR -> 1MR
Connections:
- net GND: now also R4.2, C30.2, C31.2, J2.2 (Pin_2), SW2.2, SW2.3, SW2.4, SW3.2, SW3.3, SW3.4, U4.1 (GND), U4.10 (BS0), U4.29 (VLSS), U4.30 (GND), U4.8 (VSS), U6.1 (GND), U6.10 (GND), U6.12 (GND), U7.3 (GND), U7.7 (GND); no longer C24.2, C25.2
- net SEL: now also U1.V23 (P1.03)
- net VBAT: now also J2.1 (Pin_1), U4.6 (VBAT), U6.6 (VBAT)
- net VCC: now also C31.1, U4.28 (VCC), U4.9 (VDD), U6.8 (VCC), U7.1 (OUT); no longer C25.1, C26.1, R4.1
- net VDDH: now also C30.1, U7.4 (EN), U7.6 (IN)
- net P0.18: now reaches J1.1 (Pin_1), U1.AC13 (P0.18/~{RESET})
- net P0.18: now also SW3.1
- net at C24.1: now also U4.3 (C2N)
- net P0.20: now reaches U1.AD16 (P0.20)
- net P0.20: now also U6.3 (RXD)
- net P0.22: now reaches U1.AD18 (P0.22)
- net P0.22: now also U6.2 (TXD)
- net P1.00: now reaches U1.AD22 (TRACEDATA0/P1.00)
- net P1.00: now also SW2.1
- net CW: now reaches U1.W24 (P1.02)
- net CCW: now reaches U1.Y23 (P1.01)
- new net: C26.1, U4.27 (VCOMH)
- new net: R4.1, U4.26 (IREF)
- new net: C25.1, U4.5 (C1N)
- new net: C25.2, U4.4 (C1P)
- new net: C24.2, U4.2 (C2P)
- new net SCL: U4.18 (D0)
- new net SDA: U4.12 (BS2), U4.19 (D1), U4.20 (D2)
- no-connect marks 7 -> 21
Other:
- moved on the sheet: J1
